Commit message: package sample solution
Signed-off-by: wsribunm <worawissribunma@gmail.com>

File: models/nightvapor.urdf (robot description, URDF)
Before this commit: robot nvp, 1 links, 0 joints
Links:
- link base_link: geometry visual mesh filename=packages:///auav_pylon_2025/models/fullnightvapor.dae scale=5 5 5
